Commit message: denemek istiyorum gazeboyu

File: urdf/robot_core_urdf.xacro (robot description, xacro)
@@ -1,4 +1,5 @@
 <?xml version="1.0"?>
 <robot xmlns:xacro="https://www.ros.org/wiki/xacro" name="robot">
+    <xacro:include filename="inertial_macros.xacro"/>
     <material name="white">
         <color rgba="1 1 1 1"/>
@@ -28,5 +29,4 @@
                 <box size="0.3 0.3 0.15"/>
             </geometry>
-            <material name="white"/>
         </visual>
         <collision>
@@ -35,5 +35,4 @@
                 <box size="0.3 0.3 0.15"/>
             </geometry>
-            <material name="white"/>
         </collision>
     </link>
@@ -43,5 +42,5 @@
         <child link="left_wheel"/>
         <origin xyz="0 0 0.175" rpy="-${pi/2} 0 0"/>
-        <axis ="0 0 1"/>
+        <axis xyz="0 0 1"/>
     </joint>
     <link name="left_wheel">
@@ -56,5 +55,4 @@
                 <cylinder radius="0.05" length="0.04"/>
             </geometry>
-            <material name="blue"/>
         </collision>
     </link>
@@ -64,5 +62,5 @@
         <child link="right_wheel"/>
         <origin xyz="0 0 -0.175" rpy="${pi/2} 0 0"/>
-        <axis ="0 0 -1"/>
+        <axis xyz="0 0 -1"/>
     </joint>
     <link name="right_wheel">
@@ -77,5 +75,4 @@
                 <cylinder radius="0.05" length="0.04"/>
             </geometry>
-            <material name="blue"/>
         </collision>
     </link>
@@ -91,5 +88,5 @@
                 <sphere radius="0.05"/>
             </geometry>
-            <material="black"/>
+            <material name="black"/>
         </visual>
         <collision>
@@ -97,5 +94,4 @@
                 <sphere radius="0.05"/>
             </geometry>
-            <material="black"/>
         </collision>
     </link>

File: urdf/whole.urdf.xacro (robot description, xacro)
@@ -3,4 +3,5 @@
     <!-- Example Link-->
     <link name="base_link">
+        <xacro:include filename="robot_core_urdf.xacro"/>
     </link>
 </robot>
