Commit message: run ediliyor ama akü yok

File: urdf/whole_urdf.xacro (robot description, xacro)
@@ -2,4 +2,4 @@
 <robot xmlns:xacro="https://www.ros.org/wiki/xacro" name="robot">
     <!-- Example Link-->
-    <link name="base_link"></link>
+    <xacro:include filename="robot_core_urdf.xacro"/>
 </robot>
