Commit message: düzgün urdfler

File: urdf/robot_core.urdf.xacro (robot description, xacro)
@@ -8,8 +8,8 @@
     </material>
     <material name="blue">
-        <color = "0.2 0.2 1 1"/>
+        <color rgba="0.2 0.2 1 1"/>
     </material>
     <material name="black">
-        <color = "0 0 0 1">
+        <color rgba="0 0 0 1"/>
     </material>
     <!-- BASE LİNK -->
@@ -24,5 +24,5 @@
     <link name="chassis">
         <visual>
-            <origin xyz="0.15 0 0.075">
+            <origin xyz="0.15 0 0.075"/>
             <geometry>
                 <box size="0.3 0.3 0.15"/>
@@ -30,4 +30,11 @@
             <material name="white"/>
         </visual>
+        <collision>
+            <origin xyz="0.15 0 0.075"/>
+            <geometry>
+                <box size="0.3 0.3 0.15"/>
+            </geometry>
+            <material name="white"/>
+        </collision>
     </link>
     <!-- LEFT WHEEL LİNK -->
@@ -45,4 +52,10 @@
             <material name="blue"/>
         </visual>
+        <collision>
+            <geometry>
+                <cylinder radius="0.05" length="0.04"/>
+            </geometry>
+            <material name="blue"/>
+        </collision>
     </link>
     <!-- RİGHT WHEEL LİNK -->
@@ -60,4 +73,30 @@
             <material name="blue"/>
         </visual>
+        <collision>
+            <geometry>
+                <cylinder radius="0.05" length="0.04"/>
+            </geometry>
+            <material name="blue"/>
+        </collision>
+    </link>
+    <!-- CASTER WHEEL LİNK -->
+    <joint name="caster_wheel_joint" type="fixed">
+        <parent link="base_link"/>
+        <child link="caster_wheel"/>
+        <origin xyz="0.24 0 0"/>
+    </joint>
+    <link name="caster_wheel">
+        <visual>
+            <geometry>
+                <sphere radius="0.05"/>
+            </geometry>
+            <material="black"/>
+        </visual>
+        <collision>
+            <geometry>
+                <sphere radius="0.05"/>
+            </geometry>
+            <material="black"/>
+        </collision>
     </link>
 </robot>

File: urdf/whole.urdf.xacro (robot description, xacro)
@@ -2,4 +2,5 @@
 <robot xmlns:xacro="https://www.ros.org/wiki/xacro" name="robot">
     <!-- Example Link-->
-    <link name="base_link"></link>
+    <link name="base_link">
+    </link>
 </robot>

Commit message: yolladım

File: urdf/robot_core.urdf.xacro (robot description, xacro)
@@ -1,4 +1,5 @@
 <?xml version="1.0"?>
 <robot xmlns:xacro="http://www.ros.org/wiki/xacro" name="robot">
+    <xacro: include filename="inertial_macros.xacro"/>
     <material name="white">
         <color rgba="1 1 1 1" />
@@ -28,4 +29,13 @@
             <material name="white"/>
         </visual>
+        <collision>
+            <origin xyz="0.15 0 0.075"/>
+            <geometry>
+                <box size="0.3 0.3 0.15"/>
+            </geometry>
+        </collision>
+        <xacro:inertial_box mass="0.5" x="0.3" y="0.3" z="0.15">
+            <origin xyz="0.15 0 0.075" rpy="0 0 0"/>
+        </xacro:inertial_box>
     </link>
     <!-- left wheel link -->
@@ -43,4 +53,12 @@
             <material name="blue"/>
         </visual>
+        <collision>
+            <geometry>
+                <cylinder radius="0.05"  lenght="0.04"/>
+            </geometry>
+        </collision>
+        <xacro:inertial_cylinder mass="0.1" lenght="0.04" radius="0.5">
+            <origin xyz="0 0 0" rpy="0 0 0"/>
+        </xacro:inertial_cylinder>
     </link>
     <!-- right wheel link -->
@@ -58,4 +76,34 @@
             <material name="blue"/>
         </visual>
+        <collision>
+            <geometry>
+                <cylinder radius="0.05"  lenght="0.04"/>
+            </geometry>
+        </collision>
+        <xacro:inertial_cylinder mass="0.1" lenght="0.04" radius="0.5">
+            <origin xyz="0 0 0" rpy="0 0 0"/>
+        </xacro:inertial_cylinder>
     </link>
+    <!-- right wheel link -->
+        <joint name="caster_wheel_joint" type="continuous">
+            <parent link="base_link"/>
+            <child link="caster_wheel"/>
+            <origin xyz="0.24 0 0"/>
+        </joint>
+        <link name="caster_wheel">
+            <visual>
+                <geometry>
+                    <sphere radius="0.05"/>
+                </geometry>
+                <material name="black"/>
+            </visual>
+            <collision>
+                <geometry>
+                    <sphere radius="0.05"/>
+                </geometry>
+            </collision>
+            <xacro:inertial_sphere mass="0.1" radius="0.05">
+            <origin xyz="0 0 0" rpy="0 0 0"/>
+        </xacro:inertial_sphere>
+        </link>
 </robot>
