Commit message: yamuk arac

File: urdf/robot_core.xacro (robot description, xacro)
@@ -15,5 +15,22 @@
     <!-- BASE LINK -->
     <link name="base_link">
-    </link>
+    <visual>
+      <geometry>
+        <box size="0.1 0.1 0.1"/>
+      </geometry>
+      <material name="blue">
+        <color rgba="1 0.0 0.0 1"/>
+      </material>
+    </visual>
+    <collision>
+      <geometry>
+        <box size="0.1 0.1 0.1"/>
+      </geometry>
+    </collision>
+    <inertial>
+      <mass value="5.0"/>
+      <inertia ixx="0.02" ixy="0" ixz="0" iyy="0.02" iyz="0" izz="0.02"/>
+    </inertial>
+  </link>
     <!-- CHASSIS LINK -->
     <joint name="chassis_joint" type="fixed">
@@ -37,4 +54,8 @@
             <material name="white"/>
         </collision>
+        <inertial>
+      <mass value="5.0"/>
+      <inertia ixx="0.02" ixy="0" ixz="0" iyy="0.02" iyz="0" izz="0.02"/>
+    </inertial>
     </link>
     <!-- LEFT WHEEL LINK -->
@@ -58,4 +79,8 @@
             <material name="blue"/>
         </collision>
+        <inertial>
+      <mass value="5.0"/>
+      <inertia ixx="0.02" ixy="0" ixz="0" iyy="0.02" iyz="0" izz="0.02"/>
+    </inertial>
     </link>
     <!-- RIGHT WHEEL LINK -->
@@ -79,4 +104,8 @@
             <material name="blue"/>
         </collision>
+        <inertial>
+      <mass value="5.0"/>
+      <inertia ixx="0.02" ixy="0" ixz="0" iyy="0.02" iyz="0" izz="0.02"/>
+    </inertial>
     </link>
     <!-- CASTER WHEEL LINK -->
@@ -99,4 +128,8 @@
             <material name="black"/>
         </collision>
+        <inertial>
+      <mass value="5.0"/>
+      <inertia ixx="0.02" ixy="0" ixz="0" iyy="0.02" iyz="0" izz="0.02"/>
+    </inertial>
     </link>
     <gazebo>

Commit message: araçvar

File: urdf/robot_core.xacro (robot description, xacro)
@@ -15,21 +15,4 @@
     <!-- BASE LINK -->
     <link name="base_link">
-    <visual>
-      <geometry>
-        <box size="0.1 0.1 0.1"/>
-      </geometry>
-      <material name="blue">
-        <color rgba="1 0.0 0.0 1"/>
-      </material>
-    </visual>
-    <collision>
-      <geometry>
-        <box size="0.1 0.1 0.1"/>
-      </geometry>
-    </collision>
-    <inertial>
-      <mass value="5.0"/>
-      <inertia ixx="0.02" ixy="0" ixz="0" iyy="0.02" iyz="0" izz="0.02"/>
-    </inertial>
   </link>
     <!-- CHASSIS LINK -->
@@ -41,7 +24,7 @@
     <link name="chassis">
         <visual>
-            <origin xyz="0.15 0 0.075" rpy="0 0 0"/>
+            <origin xyz="0.03 0 0.075" rpy="0 0 0"/>
             <geometry>
-                <box size="0.3 0.3 0.15"/>
+                <box size="0.35 0.31 0.15"/>
             </geometry>
             <material name="white"/>
@@ -50,5 +33,5 @@
             <origin xyz="0.15 0 0.075" rpy="0 0 0"/>
             <geometry>
-                <box size="0.3 0.3 0.15"/>
+                <box size="0.35 0.31 0.15"/>
             </geometry>
             <material name="white"/>
@@ -63,5 +46,5 @@
         <parent link="base_link"/>
         <child link="left_wheel"/>
-        <origin xyz="0 0 0.175" rpy="1.5708 0 0"/> <!-- 1.5708 rad is equivalent to pi/2 -->
+        <origin xyz="0 0.175 0" rpy="1.5708 0 0"/> <!-- 1.5708 rad is equivalent to pi/2 -->
         <axis xyz="0 0 1"/>
     </joint>
@@ -80,5 +63,5 @@
         </collision>
         <inertial>
-      <mass value="5.0"/>
+      <mass value="0.5"/>
       <inertia ixx="0.02" ixy="0" ixz="0" iyy="0.02" iyz="0" izz="0.02"/>
     </inertial>
@@ -88,5 +71,5 @@
         <parent link="base_link"/>
         <child link="right_wheel"/>
-        <origin xyz="0 0 -0.175" rpy="-1.5708 0 0"/> <!-- -1.5708 rad is equivalent to -pi/2 -->
+        <origin xyz="0 -0.175 0" rpy="-1.5708 0 0"/> <!-- -1.5708 rad is equivalent to -pi/2 -->
         <axis xyz="0 0 -1"/>
     </joint>
@@ -105,5 +88,5 @@
         </collision>
         <inertial>
-      <mass value="5.0"/>
+      <mass value="0.5"/>
       <inertia ixx="0.02" ixy="0" ixz="0" iyy="0.02" iyz="0" izz="0.02"/>
     </inertial>
@@ -129,5 +112,5 @@
         </collision>
         <inertial>
-      <mass value="5.0"/>
+      <mass value="0.5"/>
       <inertia ixx="0.02" ixy="0" ixz="0" iyy="0.02" iyz="0" izz="0.02"/>
     </inertial>
