Commit message: yangın

File: urdf/robot_core.urdf (robot description, URDF)
Before this commit: robot robot, 5 links, 4 joints
Links:
- link caster_wheel: mass None -> 0.2
- link chassis: mass None -> 5.0; geometry collision box size=0.3 0.3 0.15; visual box size=1 0.3 0.15
- link left_wheel: mass None -> 0.2
- link right_wheel: mass None -> 0.2
Joints:
- joint chassis_joint: origin xyz=0.1 0 0 -> xyz=0 0 0
- joint left_wheel_joint: origin xyz=0 0 0.175 rpy=-${pi/2} 0 0 -> xyz=0 0.175 0 rpy=1.5708 0 0
- joint right_wheel_joint: origin xyz=0 0 -0.175 rpy=${pi/2} 0 0 -> xyz=0 -0.175 0 rpy=-1.5708 0 0

File: urdf/whole_urdf.xacro (robot description, xacro)
@@ -2,6 +2,4 @@
 <robot xmlns:xacro="https://www.ros.org/wiki/xacro" name="robot">
     <!-- Example Link-->
-    <link name="base_link">
-        <xacro:include filename="robot_core_urdf.xacro"/>
-    </link>
+    <xacro:include filename="robot_core_urdf.xacro"/>
 </robot>

Commit message: arac tamam

File: urdf/robot_core.urdf (robot description, URDF)
Before this commit: robot robot, 5 links, 4 joints
Links:
- removed link caster_wheel
- removed link left_wheel
- removed link right_wheel
- added link left_wheel_link, mass 0.01; collision cylinder length=0.024 radius=0.036; visual cylinder length=0.024 radius=0.036
- added link rear_wheel_link, mass 0.001; collision sphere radius=0.021; visual sphere radius=0.021
- added link right_wheel_link, mass 0.01; collision cylinder length=0.024 radius=0.036; visual cylinder length=0.024 radius=0.036
Joints:
- removed joint caster_wheel_joint
- added joint rear_castor_joint: type fixed, parent base_link, child rear_wheel_link, origin xyz=0 0 0.0 rpy=0 0 0, axis 0 1 0
- joint left_wheel_joint: axis 0 0 1 -> 0 1 0; child left_wheel -> left_wheel_link; origin xyz=0 0.175 0 rpy=1.5708 0 0 -> xyz=0 0.13 0.015 rpy=0 0 0
- joint right_wheel_joint: axis 0 0 -1 -> 0 1 0; child right_wheel -> right_wheel_link; origin xyz=0 -0.175 0 rpy=-1.5708 0 0 -> xyz=0 -0.13 0.015 rpy=0 0 0

Commit message: kopyalama koddan düzenlenmiş duvarlar

File: urdf/robot_core.urdf (robot description, URDF)
Before this commit: robot robot, 5 links, 4 joints
Links:
- removed link caster_wheel
- removed link left_wheel
- removed link right_wheel
- added link left_wheel_link, mass 0.01; collision cylinder length=0.024 radius=0.036; visual cylinder length=0.024 radius=0.036
- added link rear_wheel_link, mass 0.001; collision sphere radius=0.021; visual sphere radius=0.021
- added link right_wheel_link, mass 0.01; collision cylinder length=0.024 radius=0.036; visual cylinder length=0.024 radius=0.036
- link chassis: geometry collision box size=0.35 0.31 0.15; visual box size=0.35 0.31 0.15
Joints:
- removed joint caster_wheel_joint
- added joint rear_castor_joint: type fixed, parent base_link, child rear_wheel_link, origin xyz=0 0 0.0 rpy=0 0 0, axis 0 1 0
- joint chassis_joint: origin xyz=0 0 0 -> xyz=0.1 0 0
- joint left_wheel_joint: axis 0 0 1 -> 0 1 0; child left_wheel -> left_wheel_link; origin xyz=0 0.175 0 rpy=1.5708 0 0 -> xyz=0 0.13 0.015 rpy=0 0 0
- joint right_wheel_joint: axis 0 0 -1 -> 0 1 0; child right_wheel -> right_wheel_link; origin xyz=0 -0.175 0 rpy=-1.5708 0 0 -> xyz=0 -0.13 0.015 rpy=0 0 0

Commit message: basic lidar

File: urdf/robot_core.urdf (robot description, URDF)
Before this commit: robot robot, 5 links, 4 joints
Links:
- added link lidar_link; visual cylinder length=0.1 radius=0.04
Joints:
- added joint lidar_joint: type fixed, parent base_link, child lidar_link, origin xyz=0.25 0 0.18 rpy=0 0 0

Commit message: check

File: urdf/robot_core.urdf (robot description, URDF)
Before this commit: robot robot, 5 links, 4 joints
Links:
- link left_wheel_link: mass 0.01 -> 0.1
- link right_wheel_link: mass 0.01 -> 0.1
Joints:
- joint left_wheel_joint: origin xyz=0 0.13 0.015 rpy=0 0 0 -> xyz=0 0.13 0.018 rpy=0 0 0
- joint right_wheel_joint: origin xyz=0 -0.13 0.015 rpy=0 0 0 -> xyz=0 -0.13 0.018 rpy=0 0 0

Commit message: manuelmove

File: urdf/robot_core.urdf (robot description, URDF)
Before this commit: robot robot, 5 links, 4 joints
Links:
- added link lidar_link; visual cylinder length=0.1 radius=0.04
- link left_wheel_link: mass 0.1 -> 0.01
- link right_wheel_link: mass 0.1 -> 0.01
Joints:
- added joint lidar_joint: type fixed, parent base_link, child lidar_link, origin xyz=0.25 0 0.18 rpy=0 0 0
- joint left_wheel_joint: origin xyz=0 0.13 0.018 rpy=0 0 0 -> xyz=0 0.13 0.015 rpy=0 0 0
- joint right_wheel_joint: origin xyz=0 -0.13 0.018 rpy=0 0 0 -> xyz=0 -0.13 0.015 rpy=0 0 0

Commit message: navigation

File: urdf/robot_core.urdf (robot description, URDF)
Before this commit: robot robot, 6 links, 5 joints
Links:
- removed link lidar_link
- added link laser; visual cylinder length=0.1 radius=0.04
Joints:
- joint lidar_joint: child lidar_link -> laser

Commit message: transfer

File: urdf/robot_core.urdf (robot description, URDF)
Before this commit: robot robot, 6 links, 5 joints
Links:
- added link laser_frame
- link laser: geometry collision cylinder length=0.1 radius=0.04; visual cylinder length=0.1 radius=0.04
Joints:
- added joint lidar_frame_joint: type fixed, parent base_link, child laser_frame, origin xyz=0.25 0 0.18 rpy=0 0 0
